File: dvrk-controller-test-board.kicad_pcb (KiCad board)
At the start: 2 copper layers, 107.9 x 104.1 mm, 34 parts, among them J1 DLM1-156, U1 STNucleo-432KC, U2 LM35DT_NOPB, U3 UA9638CDR, U4 MAX6102, U5 MAX6103, U6 SFH6206-3T, U7 DS2505

Commit message: added logo
Parts:
- added G***: LOGO, dvrk:dvrk-logo, F.Cu at (102.2, 38.0)
Other:
- board text added: "1 2 3 4 5 6"
- board text added: "5V_A"
- board text added: "5V_B"
- board text added: "A B C D E F G H J K L M N"
- board text added: "P R S T U V W X Y Z a b c"
- board text added: "V_POTA"
- board text added: "V_POTB"
- board text added: "both lights should glow"
- board text added: "dVRK Controller Test Board"
- board text added: "dac"
- board text added: "heatsink overheat"
- board text added: "ref"
- board text added: "usb port"
- board text added: "v1 (Jan 2019) Johns Hopkins University https://github.com/jhu-dvrk/ dvrk-controller-test-board"
- board text added: "↑↑↑↑↑ UP ↑↑↑↑↑"

Commit message: reannotate
Parts:
- renumbered C3 to C2

Commit message: v1.1 address Peter's comments
Parts:
- added JP5: SolderJumper_2_Open, Jumper:SolderJumper-2_P1.3mm_Open_TrianglePad1.0x1.5mm, F.Cu at (101.6, 71.1)
Connections:
- J1 pad 121: Net-(J1-Pad121) -> +5V
- J1 pad 122: Net-(J1-Pad122) -> +5V
- J1 pad 123: Net-(J1-Pad123) -> +5V
- J1 pad 124: Net-(J1-Pad124) -> +5V
- J1 pad 126: Net-(J1-Pad126) -> /VCC_B
- J1 pad 127: Net-(J1-Pad127) -> /VCC_B
- J1 pad 128: Net-(J1-Pad128) -> /VCC_B
- J1 pad 136: /POT1 -> /HE1
- J1 pad 138: /HE1 -> /HE2
- J1 pad 145: /HE1 -> /HE2
- J1 pad 32: /POT1 -> /HE1
- J1 pad 34: /POT1 -> /HE1
- J1 pad 36: /HE1 -> /HE2
- J1 pad 85: /POT1 -> /HE1
- J1 pad 87: /HE1 -> /HE2
- JP1 pad 2: /POT1 -> /HE1
- JP2 pad 2: /POT1 -> /HE1
- JP3 pad 2: /HE1 -> /HE2
- JP4 pad 2: /HE1 -> /HE2
- U1 pad 25: Net-(U1-Pad25) -> /INST_1WIRE
- U7 pad 2: /INST_1WIRE -> Net-(JP5-Pad2)
Routing:
- net /HE2: track 0.00 -> 53.0 mm, vias 0 -> 3
- net /INST_1WIRE: track 23.8 -> 61.9 mm, vias 0 -> 4
- net /POT1: track 30.3 -> 0.00 mm
- net /HE1: track 55.5 -> 73.3 mm, vias 3 -> 1
- net +5V: track 108.4 -> 118.6 mm
- net /VCC_B: track 14.9 -> 22.5 mm
- net Net-(JP5-Pad2): track 0.00 -> 4.73 mm
Other:
- board text added: "SN"
- board text added: "v1.1 (Jan 2019) Johns Hopkins University https://github.com/jhu-dvrk/ dvrk-controller-test-board"
- board text removed: "v1 (Jan 2019) Johns Hopkins University https://github.com/jhu-dvrk/ dvrk-controller-test-board"
